File: Hardware/SparkFun RTK Express.sch (EAGLE design)
At the start: 121 parts, among them J13 Internal, J16 MICRO-SD-PUSH-PUSH-EXT-PIN, J17 Qwiic Right Angle, J20 FPC_12_0.5MM_BACKFLIP, J3 USB Female Type C Connector, J4 External, J5 USB Female Type C Connector, Q1 SIL2308-TP, Q2 MBT3904DW1T1, U1 74HC4052D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

Commit message: Remove post mux opto isolation. Create v10 panel.
Parts:
- removed C24, C25: 1nF, SparkFun-Capacitors:1.0NF/1000PF-0603-50V-10%
- removed C26: 0.1uF, SparkFun-Capacitors:0.1UF-0603-25V-(+80/-20%)
- removed D4, D5: BZX84C15LT3G, SparkFun-DiscreteSemi:DIODE-ZENER-BZX84C15LT3G
- removed R10, R6: 3.3k, SparkFun-Resistors:3.3KOHM-0603-1/10W-1%
- removed R11, R8: 470, SparkFun-Resistors:470OHM-0603-1/10W-1%
- removed R12, R21: 910, SparkFun-Resistors:910OHM-0603-1/10W-5%
- removed U12: HCPL-073L, SparkFun-DiscreteSemi:DUAL-OPTO_HCPL-073LSOIC-8
- FRAME3: DESIGNER (none) -> N. Seidle; REV (none) -> v10
Connections:
- removed net DIR_IN: R11.2, U12.ANODE2
- removed net DIR_ISOLATED: R21.1, U12.VOUT2, U9.A
- removed net N$35: C25.1, D4.C, R6.2, R8.1
- removed net N$37: C24.1, D5.C, R10.2, R11.1
- removed net WT_IN: R8.2, U12.ANODE1
- removed net WT_ISOLATED: R12.1, U12.VOUT1, U8.A
- net 3.3V: no longer C26.1, R12.2, R21.2, U12.VCC
- net EXT_DIR: now also U9.A; no longer R10.1
- net EXT_WT: now also U8.A; no longer R6.1
- net GND: no longer C24.2, C25.2, C26.2, D4.A, D5.A, U12.CATHODE1, U12.CATHODE2, U12.GND
Other:
- note added: "Data Port Selection"
- note added: "v10"
- note removed: "Data Output Selection"
- note removed: "High Voltage Suppression"
- note removed: "Isolation"
- note removed: "v12"
- moved on the sheet: C27, C29, U8, U9
