File: Hardware/SparkFun RTK Express Plus.brd (EAGLE design)
At the start: 68.2 x 110.1 mm, 170 parts, among them J13 Internal, J16 MICRO-SD-PUSH-PUSH-EXT-PIN, J17 Qwiic Right Angle, J3 USB Female Type C Connector, J4 External, J5 USB Female Type C Connector, Q1 SIL2308-TP, Q2 MBT3904DW1T1, U1 74HC4052D, U10 MCP73833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

Commit message: File rename
Parts:
- removed U$20, U$21: (no value), output:V100
- added R6, R8: 10k, SparkFun-Resistors:0603
- added U$1, U$18: (no value), output:V110
Connections:
- removed net ESP_3V3: R34.2
- net 3.3V: now also R34.2, R6.2, R8.2
- net EXT_DIR: now also R6.1
- net EXT_WT: now also R8.1
Routing:
- net 3.3V: track 326.7 -> 340.8 mm, vias 11 -> 12
- net EXT_WT: track 53.8 -> 54.9 mm
- net EXT_DIR: track 62.0 -> 63.1 mm
Changed lines of the file:
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@@
 <setting verticaltext="up"/>
 </settings>
-<grid distance="0.05" unitdist="inch" unit="inch" style="lines" multiple="1" display="yes" altdistance="0.005" altunitdist="inch" altunit="inch"/>
+<grid distance="1" unitdist="mm" unit="mm" style="lines" multiple="1" display="yes" altdistance="0.1" altunitdist="mm" altunit="mm"/>
 <layers>
 <layer number="1" name="Top/Horz" color="4" fill="1" visible="yes" active="yes"/>
@@
 <attribute name="VALUE" x="48.222" y="31.651" size="0.6096" layer="27" ratio="20" rot="R270"/>
 </element>
-<element name="U$20" library="output" package="V100" value="" x="35" y="97" smashed="yes"/>
-<element name="U$21" library="output" package="V100" value="" x="35" y="47" smashed="yes" rot="MR0"/>
 <element name="J1" library="SparkFun-Connectors" package="1X02_NO_SILK" value="" x="58" y="24" smashed="yes" rot="R90">
 <attribute name="NAME" x="56.603" y="22.73" size="0.6096" layer="25" font="vector" ratio="20" rot="R90"/>
@@
 <attribute name="VALUE" x="54.6" y="3" size="0.5" layer="28" rot="MR0" align="center"/>
 </element>
+<element name="R6" library="SparkFun-Resistors" package="0603" value="10k" x="58" y="33" smashed="yes">
+<attribute name="NAME" x="58" y="33.762" size="0.6096" layer="25" font="vector" ratio="20" align="bottom-center"/>
+<attribute name="PROD_ID" value="RES-00824" x="58" y="33" size="1.778" layer="27" font="vector" ratio="15" display="off"/>
+<attribute name="VALUE" x="58" y="32.238" size="0.6096" layer="27" font="vector" ratio="20" align="top-center"/>
+</element>
+<element name="R8" library="SparkFun-Resistors" package="0603" value="10k" x="58" y="29" smashed="yes">
+<attribute name="NAME" x="58" y="29.762" size="0.6096" layer="25" font="vector" ratio="20" align="bottom-center"/>
+<attribute name="PROD_ID" value="RES-00824" x="58" y="29" size="1.778" layer="27" font="vector" ratio="15" display="off"/>
+<attribute name="VALUE" x="58" y="28.238" size="0.6096" layer="27" font="vector" ratio="20" align="top-center"/>
+</element>
+<element name="U$1" library="output" package="V110" value="" x="35" y="97" smashed="yes"/>
+<element name="U$18" library="output" package="V110" value="" x="35" y="47" smashed="yes" rot="MR0"/>
 </elements>
 <signals>
@@
 <wire x1="54.07" y1="38.735" x2="36.55144375" y2="38.735" width="0.5588" layer="2"/>
 <wire x1="36.55144375" y1="38.735" x2="34.993221875" y2="40.293221875" width="0.5588" layer="2"/>
-<wire x1="52.995" y1="76.534" x2="52.995" y2="91.31" width="0.5588" layer="16"/>
+<wire x1="52.995" y1="76.534" x2="52.995" y2="80.01" width="0.5588" layer="16"/>
+<wire x1="52.995" y1="80.01" x2="52.995" y2="91.31" width="0.5588" layer="16"/>
 <wire x1="47.85" y1="90" x2="47.85" y2="91.31" width="0.5588" layer="16"/>
 <wire x1="30.555" y1="56.8" x2="28.05" y2="56.8" width="0.3048" layer="1"/>
@@
 <wire x1="23.993" y1="55.997" x2="23.99" y2="56" width="0.1778" layer="1"/>
 <wire x1="23.99" y1="56" x2="22.85" y2="56" width="0.3048" layer="1"/>
+<contactref element="R34" pad="2"/>
+<wire x1="47.84" y1="80.01" x2="52.995" y2="80.01" width="0.1778" layer="16"/>
+<contactref element="R8" pad="2"/>
+<contactref element="R6" pad="2"/>
+<wire x1="58.85" y1="33" x2="58.85" y2="30.55" width="0.1778" layer="1"/>
+<wire x1="58.85" y1="30.55" x2="58.9" y2="30.5" width="0.1778" layer="1"/>
+<wire x1="58.9" y1="30.5" x2="58.85" y2="30.45" width="0.1778" layer="1"/>
+<wire x1="58.85" y1="30.45" x2="58.85" y2="29" width="0.1778" layer="1"/>
+<wire x1="58.9" y1="30.5" x2="54.0446" y2="30.5" width="0.1778" layer="16"/>
+<wire x1="54.0246" y1="30.48" x2="54.0446" y2="30.5" width="0.1778" layer="16"/>
+<via x="58.9" y="30.5" extent="1-16" drill="0.3048"/>
 </signal>
 <signal name="GND" airwireshidden="yes">
@@
 <wire x1="41.74" y1="93.81" x2="43.238" y2="93.81" width="0.1778" layer="16"/>
 </signal>
-<signal name="ESP_3V3" class="1">
-<contactref element="R34" pad="2"/>
-</signal>
 <signal name="EXT_WT">
 <contactref element="U1" pad="2"/>
@@
 <wire x1="31.75" y1="52.4031" x2="56.4769" y2="52.4031" width="0.1778" layer="2"/>
 <contactref element="U8" pad="P2"/>
-<wire x1="54.381" y1="25.992" x2="55.329" y2="25.992" width="0.1778" layer="1"/>
-<wire x1="56.4769" y1="27.1399" x2="56.4769" y2="52.4031" width="0.1778" layer="1"/>
 <via x="56.4769" y="52.4031" extent="1-16" drill="0.3048"/>
-<wire x1="55.329" y1="25.992" x2="56.4769" y2="27.1399" width="0.1778" layer="1"/>
+<contactref element="R8" pad="1"/>
+<wire x1="54.381" y1="25.992" x2="55.075" y2="25.992" width="0.1778" layer="1"/>
+<wire x1="57.15" y1="28.067" x2="57.15" y2="29" width="0.1778" layer="1"/>
+<wire x1="55.075" y1="25.992" x2="57.15" y2="28.067" width="0.1778" layer="1"/>
+<wire x1="58" y1="31.65" x2="57.15" y2="30.8" width="0.1778" layer="1"/>
+<wire x1="57.15" y1="29" x2="57.15" y2="30.8" width="0.1778" layer="1"/>
+<wire x1="56.4769" y1="35.2231" x2="56.4769" y2="52.4031" width="0.1778" layer="1"/>
+<wire x1="58" y1="31.65" x2="58" y2="33.7" width="0.1778" layer="1"/>
+<wire x1="58" y1="33.7" x2="56.4769" y2="35.2231" width="0.1778" layer="1"/>
 </signal>
 <signal name="EXT_DIR">
@@
 <wire x1="31.825" y1="62.559" x2="31.877" y2="62.611" width="0.1778" layer="1"/>
 <contactref element="U9" pad="P2"/>
-<wire x1="54.381" y1="31.992" x2="55.614" y2="31.992" width="0.1778" layer="1"/>
-<wire x1="55.614" y1="31.992" x2="55.88" y2="32.258" width="0.1778" layer="1"/>
 <via x="55.88" y="62.738" extent="1-16" drill="0.3048"/>
-<wire x1="55.88" y1="62.738" x2="55.88" y2="32.258" width="0.1778" layer="1"/>
+<contactref element="R6" pad="1"/>
+<wire x1="54.381" y1="31.992" x2="55.3" y2="31.992" width="0.1778" layer="1"/>
+<wire x1="55.88" y1="32.572" x2="55.3" y2="31.992" width="0.1778" layer="1"/>
+<wire x1="55.88" y1="62.738" x2="55.88" y2="33" width="0.1778" layer="1"/>
+<wire x1="55.88" y1="33" x2="55.88" y2="32.572" width="0.1778" layer="1"/>
+<wire x1="57.15" y1="33" x2="55.88" y2="33" width="0.1778" layer="1"/>
 </signal>
 <signal name="ZED_WT">

Commit message: v12 PCB - remove ground plane from accelerometer. Remove old files.
Parts:
- removed U$1, U$18: (no value), output:V110
- added U$19: (no value), output:V120
Routing:
- net GND: track 18.1 -> 44.0 mm
- net 3.3V: track 340.8 -> 353.1 mm, vias 12 -> 14
Changed lines of the file:
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@@
 <layers>
 <layer number="1" name="Top/Horz" color="4" fill="1" visible="yes" active="yes"/>
-<layer number="2" name="GND/Horz" color="1" fill="3" visible="no" active="yes"/>
-<layer number="15" name="Vert" color="4" fill="6" visible="no" active="yes"/>
+<layer number="2" name="GND/Horz" color="1" fill="3" visible="yes" active="yes"/>
+<layer number="15" name="Vert" color="4" fill="6" visible="yes" active="yes"/>
 <layer number="16" name="Bottom/Vert" color="1" fill="1" visible="yes" active="yes"/>
 <layer number="17" name="Pads" color="2" fill="1" visible="yes" active="yes"/>
@@
 <attribute name="VALUE" x="58" y="28.238" size="0.6096" layer="27" font="vector" ratio="20" align="top-center"/>
 </element>
-<element name="U$1" library="output" package="V110" value="" x="35" y="97" smashed="yes"/>
-<element name="U$18" library="output" package="V110" value="" x="35" y="47" smashed="yes" rot="MR0"/>
+<element name="U$19" library="output" package="V120" value="" x="34.925" y="97.028" smashed="yes"/>
 </elements>
 <signals>
@@
 <wire x1="52.995" y1="91.31" x2="47.85" y2="91.31" width="0.5588" layer="16"/>
 <wire x1="30" y1="41.15" x2="24.1" y2="41.15" width="0.5588" layer="1"/>
-<wire x1="24.1" y1="41.15" x2="18.51" y2="35.56" width="0.5588" layer="1"/>
+<wire x1="24.1" y1="41.15" x2="21.701" y2="38.751" width="0.5588" layer="1"/>
+<wire x1="21.701" y1="38.751" x2="18.51" y2="35.56" width="0.5588" layer="1"/>
 <wire x1="18.51" y1="35.56" x2="7.207" y2="35.56" width="0.5588" layer="1"/>
 <wire x1="7.207" y1="35.56" x2="5.5" y2="37.267" width="0.5588" layer="1"/>
@@
 <wire x1="28" y1="56.85" x2="24.846" y2="56.85" width="0.3048" layer="1"/>
 <wire x1="24.846" y1="56.85" x2="23.993" y2="55.997" width="0.3048" layer="1"/>
-<wire x1="21.75" y1="53.75" x2="21.75" y2="52.324" width="0.3048" layer="1"/>
-<wire x1="21.75" y1="52.324" x2="21.75" y2="52.25" width="0.3048" layer="1"/>
-<wire x1="21.75" y1="52.25" x2="21.75" y2="51.595" width="0.3048" layer="1"/>
-<wire x1="21.15" y1="50.995" x2="21.15" y2="50" width="0.3048" layer="1"/>
-<wire x1="21.75" y1="51.595" x2="21.15" y2="50.995" width="0.3048" layer="1"/>
-<wire x1="22.25" y1="52.25" x2="21.824" y2="52.25" width="0.3048" layer="1"/>
-<wire x1="21.824" y1="52.25" x2="21.75" y2="52.324" width="0.3048" layer="1"/>
-<wire x1="21.25" y1="53.75" x2="21.75" y2="53.75" width="0.3048" layer="1"/>
 <wire x1="43.238" y1="100.16" x2="44.747" y2="100.16" width="0.5588" layer="16"/>
 <wire x1="45.057" y1="99.85" x2="46" y2="99.85" width="0.5588" layer="16"/>
@@
 <wire x1="35.864" y1="2.844" x2="42.51941875" y2="2.844" width="0.5588" layer="16"/>
 <wire x1="49.23638125" y1="2.0428" x2="55.1788" y2="2.0428" width="0.5588" layer="16"/>
-<wire x1="22.01453125" y1="54.1542" x2="22.0232" y2="54.1542" width="0.1778" layer="1"/>
-<wire x1="21.75" y1="53.75" x2="21.75" y2="53.88966875" width="0.1778" layer="1"/>
-<wire x1="21.75" y1="53.88966875" x2="22.01453125" y2="54.1542" width="0.1778" layer="1"/>
-<wire x1="22.85" y1="54.981" x2="22.85" y2="56" width="0.1778" layer="1"/>
-<wire x1="22.0232" y1="54.1542" x2="22.85" y2="54.981" width="0.1778" layer="1"/>
 <wire x1="23.993" y1="55.997" x2="23.99" y2="56" width="0.1778" layer="1"/>
 <wire x1="23.99" y1="56" x2="22.85" y2="56" width="0.3048" layer="1"/>
@@
 <wire x1="54.0246" y1="30.48" x2="54.0446" y2="30.5" width="0.1778" layer="16"/>
 <via x="58.9" y="30.5" extent="1-16" drill="0.3048"/>
-</signal>
-<signal name="GND" airwireshidden="yes">
+<wire x1="21.25" y1="53.75" x2="21.25" y2="54.778" width="0.1778" layer="1"/>
+<wire x1="21.25" y1="54.778" x2="21.336" y2="54.864" width="0.1778" layer="1"/>
+<wire x1="21.336" y1="54.864" x2="21.717" y2="54.864" width="0.1778" layer="1"/>
+<wire x1="21.717" y1="54.864" x2="22.352" y2="54.864" width="0.1778" layer="1"/>
+<wire x1="22.352" y1="54.864" x2="22.85" y2="55.362" width="0.1778" layer="1"/>
+<wire x1="22.85" y1="55.362" x2="22.85" y2="56" width="0.1778" layer="1"/>
+<wire x1="21.75" y1="53.75" x2="21.75" y2="54.831" width="0.1778" layer="1"/>
+<wire x1="21.75" y1="54.831" x2="21.717" y2="54.864" width="0.1778" layer="1"/>
+<wire x1="22.25" y1="52.25" x2="22.25" y2="51.54015" width="0.1778" layer="1"/>
+<wire x1="22.14485" y1="51.435" x2="21.717" y2="51.435" width="0.1778" layer="1"/>
+<wire x1="21.717" y1="51.435" x2="21.59" y2="51.435" width="0.1778" layer="1"/>
+<wire x1="21.59" y1="51.435" x2="21.15" y2="50.995" width="0.1778" layer="1"/>
+<wire x1="21.15" y1="50.995" x2="21.15" y2="50" width="0.1778" layer="1"/>
+<wire x1="22.25" y1="51.54015" x2="22.14485" y2="51.435" width="0.1778" layer="1"/>
+<wire x1="21.75" y1="52.25" x2="21.75" y2="51.468" width="0.1778" layer="1"/>
+<wire x1="21.75" y1="51.468" x2="21.717" y2="51.435" width="0.1778" layer="1"/>
+<wire x1="21.15" y1="50" x2="21.15" y2="48.4845" width="0.1778" layer="1"/>
+<wire x1="21.15" y1="48.4845" x2="21.209" y2="48.4255" width="0.1778" layer="1"/>
+<via x="21.209" y="48.4255" extent="1-16" drill="0.3048"/>
+<via x="21.701" y="38.751" extent="1-16" drill="0.3048"/>
+<wire x1="21.209" y1="48.4255" x2="21.209" y2="42.35315" width="0.1778" layer="16"/>
+<wire x1="21.209" y1="42.35315" x2="21.1031" y2="42.24725" width="0.1778" layer="16"/>
+<wire x1="21.1031" y1="42.24725" x2="21.1031" y2="39.3489" width="0.1778" layer="16"/>
+<wire x1="21.1031" y1="39.3489" x2="21.701" y2="38.751" width="0.1778" layer="16"/>
+</signal>
+<signal name="GND">
 <contactref element="C1" pad="2"/>
 <contactref element="R15" pad="1"/>
@@
 <wire x1="49.75" y1="101.15" x2="49.5" y2="100.9" width="0.1778" layer="1"/>
 <via x="49.5" y="100.9" extent="1-16" drill="0.3048"/>
-<via x="19.929" y="55.989" extent="1-16" drill="0.3048"/>
-<via x="24.628" y="50.02" extent="1-16" drill="0.3048"/>
+<via x="20.437" y="59.164" extent="1-16" drill="0.3048"/>
+<via x="27.549" y="48.623" extent="1-16" drill="0.3048"/>
 <via x="49.3" y="87.0911" extent="1-16" drill="0.3048"/>
 <wire x1="14.426" y1="105.07" x2="12.92" y2="105.07" width="0.1778" layer="16"/>
@@
 <via x="51.256" y="32.858" extent="1-16" drill="0.3048"/>
 <via x="51.002" y="37.303" extent="1-16" drill="0.3048"/>
+<polygon width="0.254" layer="16" pour="cutout" isolate="0.3048">
+<vertex x="17.78" y="58.42"/>
+<vertex x="26.67" y="58.42"/>
+<vertex x="26.67" y="48.26"/>
+<vertex x="17.78" y="48.26"/>
+</polygon>
+<polygon width="0.254" layer="1" pour="cutout" isolate="0.3048">
+<vertex x="17.78" y="58.42"/>
+<vertex x="26.67" y="58.42"/>
+<vertex x="26.67" y="48.26"/>
+<vertex x="17.78" y="48.26"/>
+</polygon>
+<polygon width="0.254" layer="15" pour="cutout" isolate="0.3048">
+<vertex x="17.78" y="58.42"/>
+<vertex x="26.67" y="58.42"/>
+<vertex x="26.67" y="48.26"/>
+<vertex x="17.78" y="48.26"/>
+</polygon>
+<polygon width="0.254" layer="2" pour="cutout" isolate="0.3048">
+<vertex x="17.78" y="58.42"/>
+<vertex x="26.67" y="58.42"/>
+<vertex x="26.67" y="48.26"/>
+<vertex x="17.78" y="48.26"/>
+</polygon>
+<wire x1="22.75" y1="53.75" x2="27.08" y2="53.75" width="0.1778" layer="1"/>
+<wire x1="27.08" y1="53.75" x2="27.178" y2="53.848" width="0.1778" layer="1"/>
+<wire x1="22.75" y1="53.25" x2="27.014" y2="53.25" width="0.1778" layer="1"/>
+<wire x1="27.178" y1="53.086" x2="27.014" y2="53.25" width="0.1778" layer="1"/>
+<wire x1="22.75" y1="52.75" x2="26.842" y2="52.75" width="0.1778" layer="1"/>
+<wire x1="26.842" y1="52.75" x2="27.178" y2="53.086" width="0.1778" layer="1"/>
+<wire x1="22.25" y1="53.75" x2="22.25" y2="54.127" width="0.1778" layer="1"/>
+<wire x1="22.733" y1="54.61" x2="27.051" y2="54.61" width="0.1778" layer="1"/>
+<wire x1="22.25" y1="54.127" x2="22.733" y2="54.61" width="0.1778" layer="1"/>
+<wire x1="21.15" y1="56" x2="21.15" y2="59.504" width="0.1778" layer="1"/>
+<wire x1="21.15" y1="59.504" x2="21.209" y2="59.563" width="0.1778" layer="1"/>
+<wire x1="22.85" y1="50" x2="22.85" y2="47.615" width="0.1778" layer="1"/>
+<wire x1="26.01" y1="47.25" x2="26.75" y2="47.25" width="0.1778" layer="1"/>
+<wire x1="26.75" y1="47.25" x2="27" y2="47" width="0.1778" layer="1"/>
 </signal>
 <signal name="ESP_22/SCL">
@@
 <contactref element="U13" pad="4"/>
 <contactref element="U5" pad="33"/>
-<wire x1="22.75" y1="52.25" x2="22.75" y2="51.45" width="0.1778" layer="1"/>
-<wire x1="22.75" y1="51.45" x2="22.5" y2="51.2" width="0.1778" layer="1"/>
-<via x="22.5" y="51.2" extent="1-16" drill="0.3048"/>
-<wire x1="22.5" y1="51.2" x2="19" y2="51.2" width="0.1778" layer="2"/>
+<wire x1="22.75" y1="52.25" x2="22.75" y2="51.196" width="0.1778" layer="1"/>
+<wire x1="22.75" y1="51.196" x2="22.627" y2="51.073" width="0.1778" layer="1"/>
+<via x="22.627" y="51.073" extent="1-16" drill="0.3048"/>
+<wire x1="22.627" y1="51.073" x2="19.127" y2="51.073" width="0.1778" layer="2"/>
+<wire x1="19.127" y1="51.073" x2="19" y2="51.2" width="0.1778" layer="2"/>
 <via x="19" y="51.2" extent="1-16" drill="0.3048"/>
 <wire x1="19.088" y1="58" x2="19" y2="57.912" width="0.1778" layer="2"/>
@@
 <via x="26.8" y="49.8" extent="1-16" drill="0.3048"/>
 <wire x1="29" y1="49.9" x2="26.9" y2="49.9" width="0.5588" layer="1"/>
-<wire x1="26.8" y1="49.8" x2="26.8" y2="99.946" width="0.5588" layer="15"/>
+<wire x1="26.8" y1="49.8" x2="26.8" y2="52.07" width="0.5588" layer="15"/>
+<wire x1="26.8" y1="52.07" x2="26.8" y2="99.946" width="0.5588" layer="15"/>
 <wire x1="26.8" y1="99.946" x2="22.352" y2="104.394" width="0.5588" layer="15"/>
 <wire x1="36.3001" y1="47.95" x2="35.05" y2="47.95" width="0.5588" layer="1"/>
@@
 <wire x1="24" y1="100.15" x2="24" y2="102.746" width="0.5588" layer="16"/>
 <wire x1="24" y1="102.746" x2="22.352" y2="104.394" width="0.5588" layer="16"/>
+<wire x1="26.8" y1="52.07" x2="26.8" y2="52.07" width="0.5588" layer="15"/>
 </signal>
 <signal name="ESP32_RXI">
